File: pcb/paw_right/paw_right.kicad_sch (KiCad schematic)
At the start: 0 parts

Commit message: Added right hand PCB
Parts:
- added Battery1: Conn_01x02_Socket, Connector_JST:JST_PH_S2B-PH-K_1x02_P2.00mm_Horizontal, symbol Connector:Conn_01x02_Socket
- added D1, D10, D11, D12, D13, D14, D15, D16, D17, D2, D3, D4, D5, D6, D7, D8, D9: Diode, ScottoKeebs_Components:Diode_DO-35, symbol ScottoKeebs:Placeholder_Diode
- added ONOFF1, ONOFF2, POGO1, POGO2, POGO3, POGO4, POGO5: Conn_01x01_Socket, TestPoint:TestPoint_THTPad_1.5x1.5mm_Drill0.7mm, symbol Connector:Conn_01x01_Socket
- added RESET1: Switch, Button_Switch_THT:SW_TH_Tactile_Omron_B3F-100x, symbol ScottoKeebs:Placeholder_Switch
- added S1, S10, S11, S12, S13, S14, S15, S16, S17, S2, S3, S4, S5, S6, S7, S8, S9: Keyswitch, ScottoKeebs_Hotswap:Hotswap_Choc_V1V2, symbol ScottoKeebs:Placeholder_Keyswitch
- added U1: Nice_Nano_V2, ScottoKeebs_MCU:Nice_Nano_V2, symbol MentalDesk:MCU_Nice_Nano_V2_No_Debug
Connections:
- new net: D6.2 (A), S6.2
- new net: D2.2 (A), S2.2
- new net: D5.2 (A), S5.2
- new net: D17.2 (A), S17.2
- new net: D9.2 (A), S9.2
- new net: D11.2 (A), S11.2
- new net: D8.2 (A), S8.2
- new net: D12.2 (A), S12.2
- new net: D3.2 (A), S3.2
- new net: D1.2 (A), S1.2
- new net: D16.2 (A), S16.2
- new net: D13.2 (A), S13.2
- new net: D15.2 (A), S15.2
- new net: D10.2 (A), S10.2
- new net: D4.2 (A), S4.2
- new net: D7.2 (A), S7.2
- new net: D14.2 (A), S14.2
- new net 3V3: POGO3.1 (Pin_1), U1.21 (3.3v)
- new net B+: ONOFF1.1 (Pin_1), U1.24 (B+)
- new net Col 5: S10.1, S15.1, S17.1, S5.1, U1.14 (16)
- new net Col 6: S14.1, S16.1, S4.1, S9.1, U1.15 (14)
- new net Col 7: S13.1, S3.1, S8.1, U1.16 (15)
- new net Col 8: S12.1, S2.1, S7.1, U1.17 (18)
- new net Col 9: S1.1, S11.1, S6.1, U1.18 (19)
- new net GND: Battery1.1 (Pin_1), POGO2.1 (Pin_1), RESET1.2, U1.23 (GND), U1.3 (GND), U1.4 (GND)
- new net ONOFF: Battery1.2 (Pin_2), ONOFF2.1 (Pin_1)
- new net RDY: POGO1.1 (Pin_1), U1.7 (4)
- new net RST: RESET1.1, U1.22 (RST)
- new net Row 0: D1.1 (K), D2.1 (K), D3.1 (K), D4.1 (K), D5.1 (K), U1.8 (5)
- new net Row 1: D10.1 (K), D6.1 (K), D7.1 (K), D8.1 (K), D9.1 (K), U1.9 (6)
- new net Row 2: D11.1 (K), D12.1 (K), D13.1 (K), D14.1 (K), D15.1 (K), U1.10 (7)
- new net Row 3: D16.1 (K), D17.1 (K), U1.11 (8)
- new net SCL: POGO4.1 (Pin_1), U1.6 (3)
- new net SDA: POGO5.1 (Pin_1), U1.5 (2)
